File: Hardware/MAVRIC_Camera.sch (KiCad schematic (older format))
At the start: 61 parts, among them J1 MASTER, J2 CAMERA, J3 SERVO, J4 ICSP-PIC, J5 USB_MINI, SW1 PRGM, SW2 RESET, U1 PIC32MX250F128D, U2 MPU9150, U3 AOZ1031, U4 AOZ1031, U5 AOZ1031, X1 8MHz

Commit message: Add compensation resistor values
Parts:
- R11: value R -> 100k
- R15: value R -> 33k
- R3: value R -> 68k
Changed lines of the file:
@@
 P 7000 5850
 F 0 "R3" H 7000 5950 60  0000 C CNN
-F 1 "R" H 7000 5850 60  0000 C CNN
+F 1 "68k" H 7000 5850 60  0000 C CNN
 F 2 "~" H 7000 5850 60  0000 C CNN
 F 3 "~" H 7000 5850 60  0000 C CNN
@@
 P 6800 3550
 F 0 "R11" H 6800 3650 60  0000 C CNN
-F 1 "R" H 6800 3550 60  0000 C CNN
+F 1 "100k" H 6800 3550 60  0000 C CNN
 F 2 "~" H 6800 3550 60  0000 C CNN
 F 3 "~" H 6800 3550 60  0000 C CNN
@@
 P 7200 1450
 F 0 "R15" H 7200 1550 60  0000 C CNN
-F 1 "R" H 7200 1450 60  0000 C CNN
+F 1 "33k" H 7200 1450 60  0000 C CNN
 F 2 "~" H 7200 1450 60  0000 C CNN
 F 3 "~" H 7200 1450 60  0000 C CNN
